Commit message: Rename folder and add dependencies

File: go2_description/urdf/leg.xacro (robot description, xacro)
@@ -1,5 +1,5 @@
 <?xml version="1.0"?>
 <robot xmlns:xacro="http://www.ros.org/wiki/xacro">
-    <!-- <xacro:include filename="$(find unitree_go2_description)/transmission.xacro"/> -->
+    <!-- <xacro:include filename="$(find go2_description)/transmission.xacro"/> -->
     <xacro:macro name="leg" params="name mirror mirror_dae front_hind front_hind_dae">
         <joint name="${name}_hip_joint" type="revolute">
@@ -42,5 +42,5 @@
                 </xacro:if>
                 <geometry>
-                    <mesh filename="file://$(find unitree_go2_description)/meshes/hip.dae" scale="1 1 1"/>
+                    <mesh filename="file://$(find go2_description)/meshes/hip.dae" scale="1 1 1"/>
                 </geometry>
                 <!-- <material name="orange"/> -->
@@ -74,8 +74,8 @@
                 <geometry>
                     <xacro:if value="${mirror_dae == True}">
-                        <mesh filename="file://$(find unitree_go2_description)/meshes/thigh.dae" scale="1 1 1"/>
+                        <mesh filename="file://$(find go2_description)/meshes/thigh.dae" scale="1 1 1"/>
                     </xacro:if>
                     <xacro:if value="${mirror_dae == False}">
-                        <mesh filename="file://$(find unitree_go2_description)/meshes/thigh_mirror.dae" scale="1 1 1"/>
+                        <mesh filename="file://$(find go2_description)/meshes/thigh_mirror.dae" scale="1 1 1"/>
                     </xacro:if>
                 </geometry>
@@ -109,5 +109,5 @@
                 <origin rpy="0 0 0" xyz="0 0 0"/>
                 <geometry>
-                    <mesh filename="file://$(find unitree_go2_description)/meshes/calf.dae" scale="1 1 1"/>
+                    <mesh filename="file://$(find go2_description)/meshes/calf.dae" scale="1 1 1"/>
                 </geometry>
                 <!-- <material name="orange"/> -->

File: go2_description/urdf/lidar_4D_lidar.xacro (robot description, xacro)
@@ -11,5 +11,5 @@
             <origin rpy="0 0 0" xyz="0 0 0"/>
             <geometry>
-                <mesh filename="file://$(find unitree_go2_description)/meshes/L1_4D_Lidar.dae" scale="1 1 1"/>
+                <mesh filename="file://$(find go2_description)/meshes/L1_4D_Lidar.dae" scale="1 1 1"/>
             </geometry>
             <material name="black">
@@ -20,5 +20,5 @@
             <origin rpy="0 0 0" xyz="0 0 0"/>
             <geometry>
-                <mesh filename="file://$(find unitree_go2_description)/meshes/L1_4D_Lidar.dae" scale="1 1 1"/>
+                <mesh filename="file://$(find go2_description)/meshes/L1_4D_Lidar.dae" scale="1 1 1"/>
             </geometry>
             <material name="black">

File: go2_description/urdf/unitree_go2_gazebo.xacro (robot description, xacro)
@@ -25,5 +25,5 @@
   <gazebo>
     <plugin filename="gz_ros2_control-system" name="gz_ros2_control::GazeboSimROS2ControlPlugin">
-      <parameters>$(find unitree_go2_gazebo_sim)/config/ros_control/ros_control.yaml</parameters>
+      <parameters>$(find go2_gazebo_sim)/config/ros_control/ros_control.yaml</parameters>
       <robot_param_node>robot_state_publisher</robot_param_node>
     </plugin>

File: go2_description/urdf/unitree_go2_robot.xacro (robot description, xacro)
@@ -3,12 +3,12 @@
     xmlns:xacro="http://www.ros.org/wiki/xacro">
     <xacro:arg name="DEBUG" default="false"/>
-    <xacro:include filename="$(find unitree_go2_description)/urdf/const.xacro"/>
-    <xacro:include filename="$(find unitree_go2_description)/urdf/materials.xacro"/>
-    <xacro:include filename="$(find unitree_go2_description)/urdf/leg.xacro"/>
-    <!-- <xacro:include filename="$(find unitree_go2_description)/stairs.xacro"/> -->
-    <xacro:include filename="$(find unitree_go2_description)/urdf/unitree_go2_gazebo.xacro"/>
-    <!-- <xacro:include filename="$(find unitree_go2_description)/launch/stairs.urdf.xacro"/> -->
-    <xacro:include filename="$(find unitree_go2_description)/urdf/velodyne.xacro"/>
-    <xacro:include filename="$(find unitree_go2_description)/urdf/lidar_4D_lidar.xacro"/>
+    <xacro:include filename="$(find go2_description)/urdf/const.xacro"/>
+    <xacro:include filename="$(find go2_description)/urdf/materials.xacro"/>
+    <xacro:include filename="$(find go2_description)/urdf/leg.xacro"/>
+    <!-- <xacro:include filename="$(find go2_description)/stairs.xacro"/> -->
+    <xacro:include filename="$(find go2_description)/urdf/unitree_go2_gazebo.xacro"/>
+    <!-- <xacro:include filename="$(find go2_description)/launch/stairs.urdf.xacro"/> -->
+    <xacro:include filename="$(find go2_description)/urdf/velodyne.xacro"/>
+    <xacro:include filename="$(find go2_description)/urdf/lidar_4D_lidar.xacro"/>
     <!-- <xacro:stairs stairs="15" xpos="0" ypos="0" zpos="0" /> -->
     <!-- Rotor related joint and link is only for demonstrate location. -->
@@ -40,5 +40,5 @@
             <origin rpy="0 0 0" xyz="0 0 0"/>
             <geometry>
-                <mesh filename="file://$(find unitree_go2_description)/meshes/trunk.dae" scale="1 1 1"/>
+                <mesh filename="file://$(find go2_description)/meshes/trunk.dae" scale="1 1 1"/>
             </geometry>
         </visual>
@@ -121,5 +121,5 @@
             <origin rpy="0 0 0" xyz="0 0 0"/>
             <geometry>
-                <mesh filename="file://$(find unitree_go2_description)/meshes/L1_4D_Lidar.dae" scale="1 1 1"/>
+                <mesh filename="file://$(find go2_description)/meshes/L1_4D_Lidar.dae" scale="1 1 1"/>
             </geometry>
             <material name="black">
@@ -130,5 +130,5 @@
             <origin rpy="0 0 0" xyz="0 0 0"/>
             <geometry>
-                <mesh filename="file://$(find unitree_go2_description)/meshes/L1_4D_Lidar.dae" scale="1 1 1"/>
+                <mesh filename="file://$(find go2_description)/meshes/L1_4D_Lidar.dae" scale="1 1 1"/>
             </geometry>
             <material name="black">

File: go2_description/urdf/velodyne.xacro (robot description, xacro)
@@ -14,10 +14,10 @@
         <visual>
             <geometry>
-                <mesh filename="file://$(find unitree_go2_description)/meshes/VLP16_base_1.dae"/>
+                <mesh filename="file://$(find go2_description)/meshes/VLP16_base_1.dae"/>
             </geometry>
         </visual>
         <visual>
             <geometry>
-                <mesh filename="file://$(find unitree_go2_description)/meshes/VLP16_base_2.dae"/>
+                <mesh filename="file://$(find go2_description)/meshes/VLP16_base_2.dae"/>
             </geometry>
         </visual>
@@ -43,5 +43,5 @@
             <origin xyz="0 0 -0.0377"/>
             <geometry>
-                <mesh filename="file://$(find unitree_go2_description)/meshes/VLP16_scan.dae"/>
+                <mesh filename="file://$(find go2_description)/meshes/VLP16_scan.dae"/>
             </geometry>
         </visual>
